File: pcb/light-diffusion/light-diffusion.kicad_pcb (KiCad board)
At the start: 2 copper layers, 5 x 8 mm, 1 part

Commit message: Invert light diffusion board logo, fix lib table
Parts:
- G***: footprint feeder:logo-mask -> feeder:logo-mask-inverted
Routing:
- added copper zone on B.Cu, net (none)
- added copper zone on F.Cu, net (none)
