File: pcb/feederFloor/feederFloor.kicad_pcb (KiCad board)
At the start: 2 copper layers, 13.4 x 31.1 mm, 6 parts, among them J1 IDC, J2 Conn_01x05_Female, U1 DS28E07

Commit message: Update feeder floor, Add silkscreen for hand labeling, Fix design rules
Other:
- rule pad_to_mask_clearance: 0.051 -> 0
